Commit message: chore(config): save Rviz2 configuration file

File: ros2_ws/src/differential_robot_description/urdf/differential_robot.urdf.xacro (robot description, xacro)
@@ -2,7 +2,14 @@
 <robot xmlns:xacro="http://www.ros.org/wiki/xacro"
        name="differential_robot">
+    <!-- Robot dimensions -->
     <xacro:property name="body_length" value="0.5"/>
     <xacro:property name="body_width" value="0.4"/>
     <xacro:property name="body_height" value="0.3"/>
+    <!-- Wheel dimensions -->
+    <xacro:property name="wheel_radius" value="0.05"/>
+    <xacro:property name="wheel_width" value="0.02"/>
+    <xacro:property name="wheel_separation" value="${body_width}"/>
+    <!-- Constants -->
+    <!-- Body -->
     <link name="base_link">
         <visual>
@@ -12,3 +19,39 @@
         </visual>
     </link>
+    <!-- Front Left Wheel -->
+    <link name="front_left_wheel_link">
+        <visual>
+            <origin xyz="0 0 0" rpy="${pi/2} 0 0"/>
+            <geometry>
+                <cylinder radius="${wheel_radius}"
+                          length="${wheel_width}"/>
+            </geometry>
+        </visual>
+    </link>
+    <!-- Front Left Wheel Joint -->
+    <joint name="front_left_wheel_joint" type="continuous">
+        <parent link="base_link"/>
+        <child link="front_left_wheel_link"/>
+        <origin xyz="0 ${-wheel_separation/2} 0"
+                rpy="0 0 0"/>
+        <axis xyz="0 1 0"/>
+    </joint>
+    <!-- Front Right Wheel -->
+    <link name="front_right_wheel_link">
+        <visual>
+            <origin xyz="0 0 0" rpy="${pi/2} 0 0"/>
+            <geometry>
+                <cylinder radius="${wheel_radius}"
+                          length="${wheel_width}"/>
+            </geometry>
+        </visual>
+    </link>
+    <!-- Front Right Wheel Joint -->
+    <joint name="front_right_wheel_joint" type="continuous">
+        <parent link="base_link"/>
+        <child link="front_right_wheel_link"/>
+        <origin xyz="0 ${wheel_separation/2} 0"
+                rpy="0 0 0"/>
+        <axis xyz="0 1 0"/>
+    </joint>
 </robot>

Commit message: feat(urdf): change the description of differential robot model

File: ros2_ws/src/differential_robot_description/urdf/differential_robot.urdf.xacro (robot description, xacro)
@@ -5,8 +5,8 @@
     <xacro:property name="body_length" value="0.5"/>
     <xacro:property name="body_width" value="0.4"/>
-    <xacro:property name="body_height" value="0.3"/>
+    <xacro:property name="body_height" value="0.1"/>
     <!-- Wheel dimensions -->
-    <xacro:property name="wheel_radius" value="0.05"/>
-    <xacro:property name="wheel_width" value="0.02"/>
+    <xacro:property name="wheel_radius" value="0.125"/>
+    <xacro:property name="wheel_width" value="0.06"/>
     <xacro:property name="wheel_separation" value="${body_width}"/>
     <!-- Constants -->
@@ -33,5 +33,5 @@
         <parent link="base_link"/>
         <child link="front_left_wheel_link"/>
-        <origin xyz="0 ${-wheel_separation/2} 0"
+        <origin xyz="${body_length/2} ${-wheel_separation/2} ${body_height/2 - wheel_radius}"
                 rpy="0 0 0"/>
         <axis xyz="0 1 0"/>
@@ -51,5 +51,41 @@
         <parent link="base_link"/>
         <child link="front_right_wheel_link"/>
-        <origin xyz="0 ${wheel_separation/2} 0"
+        <origin xyz="${body_length/2} ${wheel_separation/2} ${body_height/2 - wheel_radius}"
+                rpy="0 0 0"/>
+        <axis xyz="0 1 0"/>
+    </joint>
+    <!-- Rear Left Wheel -->
+    <link name="rear_left_wheel_link">
+        <visual>
+            <origin xyz="0 0 0" rpy="${pi/2} 0 0"/>
+            <geometry>
+                <cylinder radius="${wheel_radius}"
+                            length="${wheel_width}"/>
+            </geometry>
+        </visual>
+    </link>
+    <!-- Rear left Wheel Joint -->
+    <joint name="rear_left_wheel_joint" type="continuous">
+        <parent link="base_link"/>
+        <child link="rear_left_wheel_link"/>
+        <origin xyz="${-body_length/2} ${-wheel_separation/2} ${body_height/2 - wheel_radius}"
+                rpy="0 0 0"/>
+        <axis xyz="0 1 0"/>
+    </joint>
+    <!-- Rear Right Wheel -->
+    <link name="rear_right_wheel_link">
+        <visual>
+            <origin xyz="0 0 0" rpy="${pi/2} 0 0"/>
+            <geometry>
+                <cylinder radius="${wheel_radius}"
+                            length="${wheel_width}"/>
+            </geometry>
+        </visual>
+    </link>
+    <!-- Rear Right Wheel Joint -->
+    <joint name="rear_right_wheel_joint" type="continuous">
+        <parent link="base_link"/>
+        <child link="rear_right_wheel_link"/>
+        <origin xyz="${-body_length/2} ${wheel_separation/2} ${body_height/2 - wheel_radius}"
                 rpy="0 0 0"/>
         <axis xyz="0 1 0"/>
