Commit message: fix(xacro): provide seeparate xacro files for differential and Ackermann models

File: ros2_ws/src/differential_robot_description/urdf/ackermann_robot.urdf.xacro (robot description, xacro)
@@ -18,5 +18,5 @@
         </visual>
     </link>
-     <!-- Front Left Wheel -->
+    <!-- Front Left Wheel -->
     <link name="front_left_wheel_link">
         <visual>
@@ -32,5 +32,5 @@
         <parent link="base_link"/>
         <child link="front_left_wheel_link"/>
-        <origin xyz="0 ${wheel_separation/2} ${body_height/2 - wheel_radius}"
+        <origin xyz="${body_length/2} ${wheel_separation/2} ${body_height/2 - wheel_radius}"
                 rpy="0 0 0"/>
         <axis xyz="0 1 0"/>
@@ -50,11 +50,9 @@
         <parent link="base_link"/>
         <child link="front_right_wheel_link"/>
-        <origin xyz="0 ${-wheel_separation/2} ${body_height/2 - wheel_radius}"
+        <origin xyz="${body_length/2} ${-wheel_separation/2} ${body_height/2 - wheel_radius}"
                 rpy="0 0 0"/>
         <axis xyz="0 1 0"/>
     </joint>
-</robot>
-<!--
-        <!-- Rear Left Wheel -->
+    <!-- Rear Left Wheel -->
     <link name="rear_left_wheel_link">
         <visual>
@@ -70,5 +68,5 @@
         <parent link="base_link"/>
         <child link="rear_left_wheel_link"/>
-        <origin xyz="${-body_length/2} ${-wheel_separation/2} ${body_height/2 - wheel_radius}"
+        <origin xyz="${-body_length/2} ${wheel_separation/2} ${body_height/2 - wheel_radius}"
                 rpy="0 0 0"/>
         <axis xyz="0 1 0"/>
@@ -88,7 +86,7 @@
         <parent link="base_link"/>
         <child link="rear_right_wheel_link"/>
-        <origin xyz="${-body_length/2} ${wheel_separation/2} ${body_height/2 - wheel_radius}"
+        <origin xyz="${-body_length/2} ${-wheel_separation/2} ${body_height/2 - wheel_radius}"
                 rpy="0 0 0"/>
         <axis xyz="0 1 0"/>
     </joint>
-    -->
+</robot>
